File: electronics/cm4_drone/cm4_drone.kicad_sch (KiCad schematic)
At the start: 56 parts, among them J2 HDMI_A, J8 Conn_01x02_Female, J9 Conn_01x02_Female, U1 74LVC1G04, U3 ADS1115IDGS, U4 USB2514B_Bi, U6 TPS22948DCKR

Commit message: wip new pcb with m2 connector
Parts:
- removed PWM4, PWM5, PWM6, PWM7: Conn_01x02_Female, cm4_drone:Breakout_1x02_2mm_SMD, symbol Connector:Conn_01x02_Female
- added J3: Bus_M.2_Socket_B, footprints:AMPHENOL_MDT420B03002, symbol Connector:Bus_M.2_Socket_B
- added PWM4, PWM5, PWM6, PWM7: Conn_01x03_Female, Connector_PinHeader_2.54mm:PinHeader_1x03_P2.54mm_Vertical, symbol Connector:Conn_01x03_Female
- TV1: footprint cm4_drone:Breakout_1x02_2mm_SMD -> Connector_Coaxial:U.FL_Hirose_U.FL-R-SMT-1_Vertical
- USB1: footprint cm4_drone:Breakout_1x04_2mm_SMD -> Connector_JST:JST_GH_SM04B-GHS-TB_1x04-1MP_P1.25mm_Horizontal
Connections:
- net GND: now also RADIO2.16 (DIO2), TV1.2 (Pin_2), J3.11 (GND), J3.27 (GND), J3.3 (GND), J3.33 (GND), J3.39 (GND), J3.45 (GND), J3.5 (GND), J3.51 (GND), J3.57 (GND), J3.71 (GND), J3.73 (GND), PWM4.3 (Pin_3), PWM5.3 (Pin_3), PWM6.3 (Pin_3), PWM7.3 (Pin_3); no longer TV1.1 (Pin_1)
- net I2C1_SCL: now also J3.40 (GPIO_0)
- net I2C1_SDA: now also J3.42 (GPIO_1)
- net SOFT_PWM4: now also PWM4.1 (Pin_1)
- net SOFT_PWM5: now also PWM5.1 (Pin_1)
- net SOFT_PWM6: now also PWM6.1 (Pin_1)
- net SOFT_PWM7: now also PWM7.1 (Pin_1)
- net TVOUT: now also TV1.1 (Pin_1); no longer TV1.2 (Pin_2)
- net USB2_D+: now also J3.7 (USB_D+)
- net USB2_D-: now also J3.9 (USB_D-)
- new net 3.3V: J3.2 (3.3V), J3.4 (3.3V), J3.70 (3.3V), J3.72 (3.3V), J3.74 (3.3V)
- new net PCIe_CLK_N: J3.53 (REFCLKn)
- new net PCIe_CLK_P: J3.55 (REFCLKp)
- new net PCIe_REQ: J3.52 (~{CLKREQ})
- new net PCIe_RST: J3.50 (~{PERST})
- new net PCIe_RX_N: J3.41 (PERn0/SATA-B+)
- new net PCIe_RX_P: J3.43 (PERp0/SATA-B-)
- new net PCIe_TX_N: J3.47 (PETn0/SATA-A-)
- new net PCIe_TX_P: J3.49 (PETp0/SATA-A+)
- no-connect marks 32 -> 36
Other:
- moved on the sheet: C1, SD1
